File: MCP23017.kicad_sch (KiCad schematic)
At the start: 29 parts, among them J10 Conn_PH_01x10, J2 Carte_Relais, J3 Conn_03x08_Odd_Even, J5 Conn_03x08_Odd_Even, J8 Conn_PH_01x10, J9 Conn_03x08_Odd_Even, U2 MCP23017, U3 MCP23017, U4 ULN2803ADWR

Commit message: 26/06/2025  8:54 Signed-off-by: TEST-BANC <TEST-BANC@DOMOMICRON.LOCAL>
Connections:
- net A0 is gone; now on net A01: U2.17 (A2)
- net A1 is gone; now on net A11: U2.16 (A1)
- net A2 is gone; now on net A21: U2.15 (A0)
- net SCK: no longer U2.12 (SCK)
- new net SCL: U2.12 (SCK)

Commit message: 26/06/2025  11:50 Signed-off-by: TEST-BANC <TEST-BANC@DOMOMICRON.LOCAL>
Connections:
- net GND_MCP is gone; now on net GNDD: J10.10 (Pin_10), J2.19 (Pin_19), J2.20 (Pin_20), J5.2 (Pin_2), J5.6 (Pin_6), J8.10 (Pin_10), J9.6 (Pin_6), U3.10 (VSS), U4.9 (GND)
- net SCK is gone; now on net SCL: U3.12 (SCK)
- net VCC is gone; now on net +5V: J9.1 (Pin_1)
- net +3V3 renamed +3.3V
- net GND renamed GNDD
