File: Relais.kicad_sch (KiCad schematic)
At the start: 3 parts, among them J12 Conn_01x05_P2.54mm_pinheader_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, J53 Conn_01x06_P2.54mm_pinheader_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

Commit message: 26/06/2025  11:50 Signed-off-by: TEST-BANC <TEST-BANC@DOMOMICRON.LOCAL>
Connections:
- net GND_TS3A: no longer J11.8 (GND), J12.5 (Pin_5), J53.1 (Pin_1)
- net +3V3 renamed +3.3V
- new net GNDPWR: J11.8 (GND), J12.5 (Pin_5), J53.1 (Pin_1)

Commit message: 26/06/2025  14:23 Signed-off-by: TEST-BANC <TEST-BANC@DOMOMICRON.LOCAL>
Parts:
- J11: value ~ -> TMUX1574; footprint (none) -> OmiEntreeSortie:TMUX1574; Distributeur1 (none) -> DK:296-53444-2-ND; Distributeur2 (none) -> M:595-TMUX1574PWR; Fabreference (none) -> TMUX1574PWR; Fabriquant  (none) -> Texas Instruments; Omicron (none) -> NC
Changed lines of the file:
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@@
 			)
 		)
-		(property "Value" "~"
+		(property "Value" "TMUX1574"
 			(at 125.095 45.72 0)
 			(effects
@@
 			)
 		)
-		(property "Footprint" ""
+		(property "Footprint" "OmiEntreeSortie:TMUX1574"
 			(at 120.65 50.8 0)
 			(effects
@@
 			)
 		)
-		(property "Datasheet" ""
+		(property "Datasheet" "https://www.ti.com/general/docs/suppproductinfo.tsp?distId=10&gotoUrl=https%3A%2F%2Fwww.ti.com%2Flit%2Fgpn%2Ftmux1574"
 			(at 120.65 50.8 0)
 			(effects
@@
 			)
 		)
-		(property "Description" ""
+		(property "Description" "IC SWITCH SPDTX4 4.5OHM 16TSSOP"
 			(at 120.65 50.8 0)
 			(effects
@@
 			)
 		)
-		(property "Fabriquant " ""
+		(property "Fabriquant " "Texas Instruments"
 			(at 120.65 50.8 0)
 			(effects
@@
 			)
 		)
-		(property "Fabreference" ""
+		(property "Fabreference" "TMUX1574PWR"
 			(at 120.65 50.8 0)
 			(effects
@@
 			)
 		)
-		(property "Omicron" ""
+		(property "Omicron" "NC"
 			(at 120.65 50.8 0)
 			(effects
@@
 			)
 		)
-		(property "Distributeur1" ""
+		(property "Distributeur1" "DK:296-53444-2-ND"
 			(at 120.65 50.8 0)
 			(effects
@@
 			)
 		)
-		(property "Distributeur2" ""
+		(property "Distributeur2" "M:595-TMUX1574PWR"
 			(at 120.65 50.8 0)
 			(effects
