File: alimentation.kicad_sch (KiCad schematic)
At the start: 27 parts

Commit message: version 26/06/2025 08:31
Signed-off-by: TEST-BANC <TEST-BANC@DOMOMICRON.LOCAL>
Parts:
- added C12, C13, C14: C, symbol Device:C
- added C15, C16, C17: C_Polarized, symbol Device:C_Polarized
- added J13: ~, symbol Omialimentation:TEN8_1223
- added J4: Conn_01x02, Connector_Phoenix_MC_HighVoltage:PhoenixContact_MCV_1,5_2-G-5.08_1x02_P5.08mm_Vertical, symbol Connector_Generic:Conn_01x02
- added J54: Conn_01x05_P2.54mm_pinheader_vertical, Omiconnecteur:PinHeader_1x05_P2.54mm_V_omi, symbol Omiconnecteur:Conn_01x05_P2.54mm_pinheader_vertical
- added J6: Con_01x03, Omiconnecteur:PinHeader_1x02_P2.54mm_V_omi, symbol Omiconnecteur:Conn_01x02_P2.54mm_pinheader_vertical
- added Pt10, Pt11, Pt12, Pt13, Pt14, Pt15, Pt5, Pt6, Pt7, Pt8, Pt9: PT_cms_1.0mm, Omidivers:Pt_trad_1.0mm, symbol Omidivers:PT_trad_1.0mm
- added R23, R24, R25, R26: R, symbol Device:R
- added U1: WX-DC12003, Omievalboard:WX-DC12003, symbol Omievalboard:Omi_WX-DC12003
- L7805CV1: Distributeur1 (none) -> RS: 918-1971; Distributeur2 (none) -> F : 9756078; Fabreference (none) -> L7805CV; Fabriquant (none) -> STMicroelectronics
- LM317_1, LM317_2, LM317_3: Distributeur1 (none) -> D:LM317HVT/NOPB-ND; Distributeur2 (none) -> M:926-LM317HVT/NOPB; Fabreference (none) -> LM317HVT/NOPB; Fabriquant (none) -> Texas Instruments; Omicron (none) -> 1564497
- R7, R8, R9: value 240 -> NC
Connections:
- net +11V: now also J54.3 (Pin_3), Pt5.1 (Pin_1)
- net +14V: now also J54.2 (Pin_2), Pt13.1 (Pin_1)
- net +16V: now also C12.1, C15.1, J13.22 (V+), J13.23 (V+), J54.1 (Pin_1)
- net +5V: now also J4.1 (Pin_1), J4.2 (Pin_2), J6.2 (Pin_2), Pt14.1 (Pin_1), Pt15.1 (Pin_1), U1.1 (L), U1.2 (N)
- net +8V: now also J54.4 (Pin_4), Pt6.1 (Pin_1)
- net GND renamed GND_ALIM
- net GND_ALIM: now also C12.2, C15.2, J13.2 (V-), J13.3 (V-), J54.5 (Pin_5), Pt7.1 (Pin_1), Pt8.1 (Pin_1), Pt9.1 (Pin_1)
- new net: J6.1 (Pin_1), U1.3 (OUT+)
- new net +15V: C13.1, C16.1, J13.14 (+Vout), Pt11.1 (Pin_1), R23.1, R24.1
- new net -15V: C14.2, C17.2, J13.11 (-Vout), Pt12.1 (Pin_1), R25.2, R26.2
- new net GND_220: U1.4 (OUT-)
- new net GND_TEN8: C13.2, C14.1, C16.2, C17.1, J13.16 (COM), J13.9 (COM), Pt10.1 (Pin_1), R23.2, R24.2, R25.1, R26.1
Other:
- note added: "+15V -15V"
- note added: "16V to 11V"
- note added: "16V to 14V"
- note added: "16V to 5V"
- note added: "16V to 8V"
- note added: "220 TO 5V"
- moved on the sheet: C1, C10, C11, C2, C3, C4, C5, C6, C7, C8, C9, D1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

Commit message: 26/06/2025  8:54 Signed-off-by: TEST-BANC <TEST-BANC@DOMOMICRON.LOCAL>
Connections:
- net GND_ALIM: now also J13.1 (NC)
Changed lines of the file:
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@@
+	(wire
+		(pts
+			(xy 154.94 104.14) (xy 152.4 104.14)
+		)
+		(stroke
+			(width 0)
+			(type default)
+		)
+	)
 	(wire
 		(pts
@@
 		(pts
 			(xy 55.88 38.1) (xy 60.96 38.1)
+		)
+		(stroke
+			(width 0)
+			(type default)
+		)
+	)
+	(wire
+		(pts
+			(xy 152.4 104.14) (xy 152.4 105.41)
 		)
 		(stroke
@@
 			(effects
 				(font
+					(size 1.27 1.27)
+				)
+				(justify right)
+				(hide yes)
+			)
+		)
+	)
+	(global_label "GND_ALIM"
+		(shape input)
+		(at 152.4 105.41 270)
+		(fields_autoplaced yes)
+		(effects
+			(font
+				(size 1.27 1.27)
+			)
+			(justify right)
+		)
+		(property "Intersheetrefs" "${INTERSHEET_REFS}"
+			(at 152.4 117.4062 90)
+			(effects
+				(font

Commit message: 26/06/2025  11:50 Signed-off-by: TEST-BANC <TEST-BANC@DOMOMICRON.LOCAL>
Parts:
- removed J4: Conn_01x02, Connector_Phoenix_MC_HighVoltage:PhoenixContact_MCV_1,5_2-G-5.08_1x02_P5.08mm_Vertical, symbol Connector_Generic:Conn_01x02
- removed J6: Con_01x03, Omiconnecteur:PinHeader_1x02_P2.54mm_V_omi, symbol Omiconnecteur:Conn_01x02_P2.54mm_pinheader_vertical
- removed Pt15: PT_cms_1.0mm, Omidivers:Pt_trad_1.0mm, symbol Omidivers:PT_trad_1.0mm
- removed U1: WX-DC12003, Omievalboard:WX-DC12003, symbol Omievalboard:Omi_WX-DC12003
Connections:
- net GND_ALIM renamed GNDPWR
Other:
- note removed: "220 TO 5V"

Commit message: 26/06/2025  14:23 Signed-off-by: TEST-BANC <TEST-BANC@DOMOMICRON.LOCAL>
Parts:
- J13: footprint (none) -> Omialimentation:CONV_TEN_8-1223; Distributeur1 (none) -> RS:423-9628P; Distributeur2 (none) -> F: 1205021; Fabreference (none) -> TEN 8-1223; Fabriquant  (none) -> TRACOPOWER; Omicron (none) -> NC
Changed lines of the file:
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@@
 			)
 		)
-		(property "Footprint" ""
+		(property "Footprint" "Omialimentation:CONV_TEN_8-1223"
 			(at 163.83 95.25 0)
 			(effects
@@
 			)
 		)
-		(property "Datasheet" ""
+		(property "Datasheet" "https://docs.rs-online.com/3545/0900766b816e9de6.pdf"
 			(at 163.83 95.25 0)
 			(effects
@@
 			)
 		)
-		(property "Description" ""
+		(property "Description" "Convertisseur DC-DC TRACOPOWER TEN 8, Montage traversant, 8W, 2 sorties, ±15V c.c., ±265mA"
 			(at 163.83 95.25 0)
 			(effects
 				(font
+					(size 1.27 1.27)
+				)
+				(hide yes)
+			)
+		)
+		(property "Fabriquant " "TRACOPOWER"
+			(at 163.83 109.728 0)
+			(effects
+				(font
+					(size 1.27 1.27)
+				)
+				(hide yes)
+			)
+		)
+		(property "Fabreference" "TEN 8-1223"
+			(at 164.338 109.474 0)
+			(effects
+				(font
+					(size 1.27 1.27)
+				)
+				(hide yes)
+			)
+		)
+		(property "Omicron" "NC"
+			(at 164.084 109.474 0)
+			(effects
+				(font
+					(size 1.27 1.27)
+				)
+				(hide yes)
+			)
+		)
+		(property "Distributeur1" "RS:423-9628P"
+			(at 164.846 109.474 0)
+			(effects
+				(font
+					(size 1.27 1.27)
+				)
+				(hide yes)
+			)
+		)
+		(property "Distributeur2" "F: 1205021"
+			(at 164.592 109.474 0)
+			(effects
+				(font
